File: PCB/TS65.sch (KiCad schematic (older format))
At the start: 215 parts

Commit message: Rev 0.7
Parts:
- added BREAKHOLES3, BREAKHOLES4, BREAKHOLES5, BREAKHOLES6: MISC, prettylib:BreakHoles, symbol MISC
Other:
- moved on the sheet: BREAKHOLES1, BREAKHOLES2
Changed lines of the file:
@@
 Sheet 1 3
 Title "TS65"
-Date "2016-05-01"
-Rev "Rev 0.6"
+Date "2016-05-17"
+Rev "Rev 0.7"
 Comp "MOZ"
 Comment1 ""
@@
 L MISC BREAKHOLES2
 U 1 1 56CA654B
-P 9000 7800
-F 0 "BREAKHOLES2" H 9000 7950 60  0000 C CNN
-F 1 "MISC" H 9000 7650 60  0001 C CNN
-F 2 "prettylib:BreakHoles" H 9000 7800 60  0001 C CNN
-F 3 "" H 9000 7800 60  0000 C CNN
-	1    9000 7800
+P 8500 7800
+F 0 "BREAKHOLES2" H 8500 7950 60  0000 C CNN
+F 1 "MISC" H 8500 7650 60  0001 C CNN
+F 2 "prettylib:BreakHoles" H 8500 7800 60  0001 C CNN
+F 3 "" H 8500 7800 60  0000 C CNN
+	1    8500 7800
 	1    0    0    -1
 $EndComp
@@
 L MISC BREAKHOLES1
 U 1 1 56CA44F1
-P 9000 7350
-F 0 "BREAKHOLES1" H 9000 7500 60  0000 C CNN
-F 1 "MISC" H 9000 7200 60  0001 C CNN
-F 2 "prettylib:BreakHoles" H 9000 7350 60  0001 C CNN
-F 3 "" H 9000 7350 60  0000 C CNN
-	1    9000 7350
+P 8500 7350
+F 0 "BREAKHOLES1" H 8500 7500 60  0000 C CNN
+F 1 "MISC" H 8500 7200 60  0001 C CNN
+F 2 "prettylib:BreakHoles" H 8500 7350 60  0001 C CNN
+F 3 "" H 8500 7350 60  0000 C CNN
+	1    8500 7350
 	1    0    0    -1
 $EndComp
@@
 Wire Wire Line
 	5200 7550 4250 7550
+$Comp
+L MISC BREAKHOLES6
+U 1 1 573F8792
+P 9500 7800
+F 0 "BREAKHOLES6" H 9500 7950 60  0000 C CNN
+F 1 "MISC" H 9500 7650 60  0001 C CNN
+F 2 "prettylib:BreakHoles" H 9500 7800 60  0001 C CNN
+F 3 "" H 9500 7800 60  0000 C CNN
+	1    9500 7800
+	1    0    0    -1
+$EndComp
+$Comp
+L MISC BREAKHOLES5
+U 1 1 573F8798
+P 9500 7350
+F 0 "BREAKHOLES5" H 9500 7500 60  0000 C CNN
+F 1 "MISC" H 9500 7200 60  0001 C CNN
+F 2 "prettylib:BreakHoles" H 9500 7350 60  0001 C CNN
+F 3 "" H 9500 7350 60  0000 C CNN
+	1    9500 7350
+	1    0    0    -1
+$EndComp
+$Comp
+L MISC BREAKHOLES4
+U 1 1 573F8ABA
+P 9000 7800
+F 0 "BREAKHOLES4" H 9000 7950 60  0000 C CNN
+F 1 "MISC" H 9000 7650 60  0001 C CNN
+F 2 "prettylib:BreakHoles" H 9000 7800 60  0001 C CNN
+F 3 "" H 9000 7800 60  0000 C CNN
+	1    9000 7800
+	-1   0    0    1
+$EndComp
+$Comp
+L MISC BREAKHOLES3
+U 1 1 573F8AC0
+P 9000 7350
+F 0 "BREAKHOLES3" H 9000 7500 60  0000 C CNN
+F 1 "MISC" H 9000 7200 60  0001 C CNN
+F 2 "prettylib:BreakHoles" H 9000 7350 60  0001 C CNN
+F 3 "" H 9000 7350 60  0000 C CNN
+	1    9000 7350
+	-1   0    0    1
+$EndComp
 $EndSCHEMATC
